Commit message: work on thesis

File: pycram/resources/worlds/kitchen-small.urdf (robot description, URDF)
Before this commit: robot iai_oven_area, 77 links, 76 joints
Links:
- removed link table_area
Joints:
- removed joint table_area_joint

File: pycram/resources/worlds/kitchen.urdf (robot description, URDF)
Before this commit: robot iai_oven_area, 84 links, 83 joints
Links:
- removed link table_area_main
Joints:
- removed joint table_area_main_joint
