Commit message: luca sampling method and main merge start

File: pycram/resources/worlds/apartment.urdf (robot description, URDF)
Before this commit: robot apartment, 113 links, 112 joints
Links:
- link coffee_table: geometry collision mesh filename=package://iai_apartment/meshes/visual/coffee_table.dae; visual mesh filename=package://iai_apartment/meshes/visual/coffee_table.dae
- link table_area_main: geometry collision mesh filename=package://iai_kitchen/meshes/misc/big_table_1.obj; visual mesh filename=package://iai_kitchen/meshes/misc/big_table_1.obj
- link walls: geometry 
Joints:
- joint table_area_main_joint: origin xyz=5 4 0 rpy=0 0 1.57 -> xyz=5 4 0.3619 rpy=0 0 1.57

Commit message: fixed wiping and mixing again

File: pycram/resources/worlds/apartment.urdf (robot description, URDF)
Before this commit: robot apartment, 113 links, 112 joints
Links:
- removed link wall_coloksu_wall1
- removed link wall_coloksu_wall2
- removed link wall_coloksu_wall3
- removed link wall_coloksu_wall4
Joints:
- removed joint wall_coloksu_wall1_joint
- removed joint wall_coloksu_wall2_joint
- removed joint wall_coloksu_wall3_joint
- removed joint wall_coloksu_wall4_joint
