Commit message: g1 in single sscenariou

File: pycram/resources/worlds/isr-testbed.urdf (robot description, URDF)
Before this commit: robot world, 64 links, 63 joints
Links:
- removed link pizza_box__pizza_box__base_link
Joints:
- removed joint pizza_box__pizza_box__base_link_joint

File: pycram/resources/worlds/kitchen.urdf (robot description, URDF)
Before this commit: robot iai_oven_area, 83 links, 82 joints
Links:
- link fridge_area: geometry collision mesh filename=package://iai_kitchen/meshes/racks/FridgeArea.dae; visual mesh filename=package://iai_kitchen/meshes/racks/FridgeArea.dae
- link fridge_area_lower_drawer_handle: geometry collision mesh filename=package://iai_kitchen/meshes/handles/Handle60.dae; visual mesh filename=package://iai_kitchen/meshes/handles/Handle60.dae
- link fridge_area_lower_drawer_main: geometry collision mesh filename=package://iai_kitchen/meshes/drawers/Drawer_60_29.dae; visual mesh filename=package://iai_kitchen/meshes/drawers/Drawer_60_29.dae
- link iai_fridge_door: geometry collision mesh filename=package://iai_kitchen/meshes/misc/FridgeDoor.dae; visual mesh filename=package://iai_kitchen/meshes/misc/FridgeDoor.dae
- link iai_fridge_door_handle: geometry collision mesh filename=package://iai_kitchen/meshes/handles/VHandle90.dae; visual mesh filename=package://iai_kitchen/meshes/handles/VHandle90.dae
- link iai_fridge_main: geometry collision mesh filename=package://iai_kitchen/meshes/misc/Fridge.dae; visual mesh filename=package://iai_kitchen/meshes/misc/Fridge.dae
- link kitchen_island: geometry collision mesh filename=package://iai_kitchen/meshes/racks/IslandArea.dae; visual mesh filename=package://iai_kitchen/meshes/racks/IslandArea.dae
- link kitchen_island_left_lower_drawer_handle: geometry collision mesh filename=package://iai_kitchen/meshes/handles/Handle60.dae; visual mesh filename=package://iai_kitchen/meshes/handles/Handle60.dae
- link kitchen_island_left_lower_drawer_main: geometry collision mesh filename=package://iai_kitchen/meshes/drawers/Drawer_60_29.dae; visual mesh filename=package://iai_kitchen/meshes/drawers/Drawer_60_29.dae
- link kitchen_island_left_panel: geometry collision mesh filename=package://iai_kitchen/meshes/drawers/Panel_60.dae; visual mesh filename=package://iai_kitchen/meshes/drawers/Panel_60.dae
- link kitchen_island_left_upper_drawer_handle: geometry collision mesh filename=package://iai_kitchen/meshes/handles/Handle60.dae; visual mesh filename=package://iai_kitchen/meshes/handles/Handle60.dae
- link kitchen_island_left_upper_drawer_main: geometry collision mesh filename=package://iai_kitchen/meshes/drawers/Drawer_60_29.dae; visual mesh filename=package://iai_kitchen/meshes/drawers/Drawer_60_29.dae
- link kitchen_island_middle_lower_drawer_handle: geometry collision mesh filename=package://iai_kitchen/meshes/handles/Handle100.dae; visual mesh filename=package://iai_kitchen/meshes/handles/Handle100.dae
- link kitchen_island_middle_lower_drawer_main: geometry collision mesh filename=package://iai_kitchen/meshes/drawers/Drawer_100_29.dae; visual mesh filename=package://iai_kitchen/meshes/drawers/Drawer_100_29.dae
- link kitchen_island_middle_panel: geometry collision mesh filename=package://iai_kitchen/meshes/drawers/Panel_100.dae; visual mesh filename=package://iai_kitchen/meshes/drawers/Panel_100.dae
- link kitchen_island_middle_upper_drawer_handle: geometry collision mesh filename=package://iai_kitchen/meshes/handles/Handle100.dae; visual mesh filename=package://iai_kitchen/meshes/handles/Handle100.dae
- link kitchen_island_middle_upper_drawer_main: geometry collision mesh filename=package://iai_kitchen/meshes/drawers/Drawer_100_29.dae; visual mesh filename=package://iai_kitchen/meshes/drawers/Drawer_100_29.dae
- link kitchen_island_right_lower_drawer_handle: geometry collision mesh filename=package://iai_kitchen/meshes/handles/Handle60.dae; visual mesh filename=package://iai_kitchen/meshes/handles/Handle60.dae
- link kitchen_island_right_lower_drawer_main: geometry collision mesh filename=package://iai_kitchen/meshes/drawers/Drawer_60_29.dae; visual mesh filename=package://iai_kitchen/meshes/drawers/Drawer_60_29.dae
- link kitchen_island_right_panel: geometry collision mesh filename=package://iai_kitchen/meshes/drawers/Panel_60.dae; visual mesh filename=package://iai_kitchen/meshes/drawers/Panel_60.dae
- link kitchen_island_right_upper_drawer_handle: geometry collision mesh filename=package://iai_kitchen/meshes/handles/Handle60.dae; visual mesh filename=package://iai_kitchen/meshes/handles/Handle60.dae
- link kitchen_island_right_upper_drawer_main: geometry collision mesh filename=package://iai_kitchen/meshes/drawers/Drawer_60_29.dae; visual mesh filename=package://iai_kitchen/meshes/drawers/Drawer_60_29.dae
- link kitchen_island_stove: geometry collision mesh filename=package://iai_kitchen/meshes/misc/Stove.dae; visual mesh filename=package://iai_kitchen/meshes/misc/Stove.dae
- link oven_area_area: geometry collision mesh filename=package://iai_kitchen/meshes/racks/OvenArea.dae; visual mesh filename=package://iai_kitchen/meshes/racks/OvenArea.dae
- link oven_area_area_left_drawer_handle: geometry collision mesh filename=package://iai_kitchen/meshes/handles/VHandle130.dae; visual mesh filename=package://iai_kitchen/meshes/handles/VHandle130.dae
- link oven_area_area_left_drawer_main: geometry collision mesh filename=package://iai_kitchen/meshes/drawers/VDrawer.dae; visual mesh filename=package://iai_kitchen/meshes/drawers/VDrawer.dae
- link oven_area_area_middle_lower_drawer_handle: geometry collision mesh filename=package://iai_kitchen/meshes/handles/Handle60.dae; visual mesh filename=package://iai_kitchen/meshes/handles/Handle60.dae
- link oven_area_area_middle_lower_drawer_main: geometry collision mesh filename=package://iai_kitchen/meshes/drawers/Drawer_60_58.dae; visual mesh filename=package://iai_kitchen/meshes/drawers/Drawer_60_58.dae
- link oven_area_area_middle_upper_drawer_handle: geometry collision mesh filename=package://iai_kitchen/meshes/handles/Handle60.dae; visual mesh filename=package://iai_kitchen/meshes/handles/Handle60.dae
- link oven_area_area_middle_upper_drawer_main: geometry collision mesh filename=package://iai_kitchen/meshes/drawers/Drawer_60_14.dae; visual mesh filename=package://iai_kitchen/meshes/drawers/Drawer_60_14.dae
- link oven_area_oven_door: geometry collision mesh filename=package://iai_kitchen/meshes/oven/OvenDoor.dae; visual mesh filename=package://iai_kitchen/meshes/oven/OvenDoor.dae
- link oven_area_oven_door_handle: geometry collision mesh filename=package://iai_kitchen/meshes/handles/Handle60.dae; visual mesh filename=package://iai_kitchen/meshes/handles/Handle60.dae
- link oven_area_oven_knob_oven: geometry collision mesh filename=package://iai_kitchen/meshes/oven/Knob.dae; visual mesh filename=package://iai_kitchen/meshes/oven/Knob.dae
- link oven_area_oven_knob_stove_1: geometry collision mesh filename=package://iai_kitchen/meshes/oven/Knob.dae; visual mesh filename=package://iai_kitchen/meshes/oven/Knob.dae
- link oven_area_oven_knob_stove_2: geometry collision mesh filename=package://iai_kitchen/meshes/oven/Knob.dae; visual mesh filename=package://iai_kitchen/meshes/oven/Knob.dae
- link oven_area_oven_knob_stove_3: geometry collision mesh filename=package://iai_kitchen/meshes/oven/Knob.dae; visual mesh filename=package://iai_kitchen/meshes/oven/Knob.dae
- link oven_area_oven_knob_stove_4: geometry collision mesh filename=package://iai_kitchen/meshes/oven/Knob.dae; visual mesh filename=package://iai_kitchen/meshes/oven/Knob.dae
- link oven_area_oven_main: geometry collision mesh filename=package://iai_kitchen/meshes/oven/OvenMain.dae; visual mesh filename=package://iai_kitchen/meshes/oven/OvenMain.dae
- link oven_area_oven_panel: geometry collision mesh filename=package://iai_kitchen/meshes/oven/OvenPanel.dae; visual mesh filename=package://iai_kitchen/meshes/oven/OvenPanel.dae
- link sink_area: geometry collision mesh filename=package://iai_kitchen/meshes/racks/SinkArea.dae; visual mesh filename=package://iai_kitchen/meshes/racks/SinkArea.dae
- link sink_area_dish_washer_door: geometry collision mesh filename=package://iai_kitchen/meshes/misc/DishWasherDoor.dae; visual mesh filename=package://iai_kitchen/meshes/misc/DishWasherDoor.dae
- link sink_area_dish_washer_door_handle: geometry collision mesh filename=package://iai_kitchen/meshes/handles/Handle60.dae; visual mesh filename=package://iai_kitchen/meshes/handles/Handle60.dae
- link sink_area_dish_washer_main: geometry collision mesh filename=package://iai_kitchen/meshes/misc/DishWasher.dae; visual mesh filename=package://iai_kitchen/meshes/misc/DishWasher.dae
- link sink_area_left_bottom_drawer_handle: geometry collision mesh filename=package://iai_kitchen/meshes/handles/Handle80.dae; visual mesh filename=package://iai_kitchen/meshes/handles/Handle80.dae
- link sink_area_left_bottom_drawer_main: geometry collision mesh filename=package://iai_kitchen/meshes/drawers/Drawer_80_29.dae; visual mesh filename=package://iai_kitchen/meshes/drawers/Drawer_80_29.dae
- link sink_area_left_middle_drawer_handle: geometry collision mesh filename=package://iai_kitchen/meshes/handles/Handle80.dae; visual mesh filename=package://iai_kitchen/meshes/handles/Handle80.dae
- link sink_area_left_middle_drawer_main: geometry collision mesh filename=package://iai_kitchen/meshes/drawers/Drawer_80_29.dae; visual mesh filename=package://iai_kitchen/meshes/drawers/Drawer_80_29.dae
- link sink_area_left_upper_drawer_handle: geometry collision mesh filename=package://iai_kitchen/meshes/handles/Handle80.dae; visual mesh filename=package://iai_kitchen/meshes/handles/Handle80.dae
- link sink_area_left_upper_drawer_main: geometry collision mesh filename=package://iai_kitchen/meshes/drawers/Drawer_80_14.dae; visual mesh filename=package://iai_kitchen/meshes/drawers/Drawer_80_14.dae
- link sink_area_right_panel: geometry collision mesh filename=package://iai_kitchen/meshes/drawers/Panel_60.dae; visual mesh filename=package://iai_kitchen/meshes/drawers/Panel_60.dae
- link sink_area_sink: geometry collision mesh filename=package://iai_kitchen/meshes/misc/Sink.dae; visual mesh filename=package://iai_kitchen/meshes/misc/Sink.dae
- link sink_area_trash_drawer_handle: geometry collision mesh filename=package://iai_kitchen/meshes/handles/Handle60.dae; visual mesh filename=package://iai_kitchen/meshes/handles/Handle60.dae
- link sink_area_trash_drawer_main: geometry collision mesh filename=package://iai_kitchen/meshes/drawers/Drawer_60_58.dae; visual mesh filename=package://iai_kitchen/meshes/drawers/Drawer_60_58.dae
