Commit message: renaming pycram to cora_plex

File: cora_plex/resources/robots/ur5_robotiq.urdf (robot description, URDF)
Before this commit: robot ur5_robotiq, 20 links, 19 joints
Links:
- link base_link: geometry collision mesh filename=package://cora_plex/resources/meshes/ur5/collision/base.stl; visual mesh filename=package://cora_plex/resources/meshes/ur5/visual/base.dae
- link forearm_link: geometry collision mesh filename=package://cora_plex/resources/meshes/ur5/collision/forearm.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; visual mesh filename=package://cora_plex/resources/meshes/ur5/visual/forearm.dae
- link robotiq_85_base_link: geometry collision mesh filename=package://cora_plex/resources/meshes/robotiq/collision/robo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; visual mesh filename=package://cora_plex/resources/meshes/robotiq/visual/robotiq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
- link robotiq_85_left_finger_link: geometry collision mesh filename=package://cora_plex/resources/meshes/robotiq/collision/robo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; visual mesh filename=package://cora_plex/resources/meshes/robotiq/visual/robotiq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
- link robotiq_85_left_finger_tip_link: geometry collision mesh filename=package://cora_plex/resources/meshes/robotiq/collision/robo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; visual mesh filename=package://cora_plex/resources/meshes/robotiq/visual/robotiq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
- link robotiq_85_left_inner_knuckle_link: geometry collision mesh filename=package://cora_plex/resources/meshes/robotiq/collision/robo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; visual mesh filename=package://cora_plex/resources/meshes/robotiq/visual/robotiq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
- link robotiq_85_left_knuckle_link: geometry collision mesh filename=package://cora_plex/resources/meshes/robotiq/collision/robo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; visual mesh filename=package://cora_plex/resources/meshes/robotiq/visual/robotiq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
- link robotiq_85_right_finger_link: geometry collision mesh filename=package://cora_plex/resources/meshes/robotiq/collision/robo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; visual mesh filename=package://cora_plex/resources/meshes/robotiq/visual/robotiq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
- link robotiq_85_right_finger_tip_link: geometry collision mesh filename=package://cora_plex/resources/meshes/robotiq/collision/robo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; visual mesh filename=package://cora_plex/resources/meshes/robotiq/visual/robotiq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
- link robotiq_85_right_inner_knuckle_link: geometry collision mesh filename=package://cora_plex/resources/meshes/robotiq/collision/robo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; visual mesh filename=package://cora_plex/resources/meshes/robotiq/visual/robotiq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
- link robotiq_85_right_knuckle_link: geometry collision mesh filename=package://cora_plex/resources/meshes/robotiq/collision/robo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; visual mesh filename=package://cora_plex/resources/meshes/robotiq/visual/robotiq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
- link robotiq_coupler: geometry collision mesh filename=package://cora_plex/resources/meshes/robotiq/robotiq_85_cou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 scale=1 1 1; visual mesh filename=package://cora_plex/resources/meshes/robotiq/robotiq_85_cou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 scale=1 1 1
- link shoulder_link: geometry collision mesh filename=package://cora_plex/resources/meshes/ur5/collision/shoulder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; visual mesh filename=package://cora_plex/resources/meshes/ur5/visual/shoulder.dae
- link upper_arm_link: geometry collision mesh filename=package://cora_plex/resources/meshes/ur5/collision/upperarm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; visual mesh filename=package://cora_plex/resources/meshes/ur5/visual/upperarm.dae
- link wrist_1_link: geometry collision mesh filename=package://cora_plex/resources/meshes/ur5/collision/wrist1.s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; visual mesh filename=package://cora_plex/resources/meshes/ur5/visual/wrist1.dae
- link wrist_2_link: geometry collision mesh filename=package://cora_plex/resources/meshes/ur5/collision/wrist2.s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; visual mesh filename=package://cora_plex/resources/meshes/ur5/visual/wrist2.dae
- link wrist_3_link: geometry collision mesh filename=package://cora_plex/resources/meshes/ur5/collision/wrist3.s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; visual mesh filename=package://cora_plex/resources/meshes/ur5/visual/wrist3.dae
